Commit message: feat(m3): 完成 W1 至 W4 传感器单元基线

File: src/robot_core/ai_robot_description/urdf/ai_robot.urdf.xacro (robot description, xacro)
@@ -2,12 +2,18 @@
 <robot name="ai_robot" xmlns:xacro="http://www.ros.org/wiki/xacro">
   <xacro:arg name="model_config" default="$(find ai_robot_description)/config/robot_model.yaml"/>
+  <xacro:arg name="sensor_config" default="$(find ai_robot_description)/config/sensor_model.yaml"/>
   <xacro:arg name="enable_control" default="false"/>
+  <xacro:arg name="enable_lidar" default="false"/>
+  <xacro:arg name="enable_camera" default="false"/>
   <xacro:arg name="controller_config" default=""/>
   <xacro:property name="model_config_path" value="$(arg model_config)"/>
+  <xacro:property name="sensor_config_path" value="$(arg sensor_config)"/>
   <xacro:property name="model" value="${xacro.load_yaml(model_config_path)}"/>
+  <xacro:property name="sensors" value="${xacro.load_yaml(sensor_config_path)}"/>
   <xacro:include filename="macros/inertial.xacro"/>
   <xacro:include filename="macros/base.xacro"/>
   <xacro:include filename="macros/running_gear.xacro"/>
   <xacro:include filename="macros/control.xacro"/>
+  <xacro:include filename="macros/sensors.xacro"/>
   <xacro:base_structure model="${model}"/>
   <xacro:drive_wheel
@@ -23,4 +29,10 @@
   <xacro:support_ball item="${model['casters']['items'][0]}" casters="${model['casters']}"/>
   <xacro:support_ball item="${model['casters']['items'][1]}" casters="${model['casters']}"/>
+  <xacro:if value="$(arg enable_lidar)">
+    <xacro:lidar_sensor lidar="${sensors['lidar']}"/>
+  </xacro:if>
+  <xacro:if value="$(arg enable_camera)">
+    <xacro:camera_sensor camera="${sensors['camera']}"/>
+  </xacro:if>
   <xacro:if value="$(arg enable_control)">
     <xacro:gazebo_control controller_config="$(arg controller_config)"/>

Commit message: feat(m3): 完成 W5 IMU 单元验证

File: src/robot_core/ai_robot_description/urdf/ai_robot.urdf.xacro (robot description, xacro)
@@ -6,4 +6,5 @@
   <xacro:arg name="enable_lidar" default="false"/>
   <xacro:arg name="enable_camera" default="false"/>
+  <xacro:arg name="enable_imu" default="false"/>
   <xacro:arg name="controller_config" default=""/>
   <xacro:property name="model_config_path" value="$(arg model_config)"/>
@@ -35,4 +36,7 @@
     <xacro:camera_sensor camera="${sensors['camera']}"/>
   </xacro:if>
+  <xacro:if value="$(arg enable_imu)">
+    <xacro:imu_sensor imu="${sensors['imu']}"/>
+  </xacro:if>
   <xacro:if value="$(arg enable_control)">
     <xacro:gazebo_control controller_config="$(arg controller_config)"/>

File: src/robot_core/ai_robot_description/urdf/macros/sensors.xacro (robot description, xacro)
@@ -93,3 +93,41 @@
     </gazebo>
   </xacro:macro>
+  <xacro:macro name="imu_sensor" params="imu">
+    <link name="${imu['link_name']}">
+      <visual>
+        <geometry><box size="${' '.join(str(v) for v in imu['housing']['size'])}"/></geometry>
+        <material name="ai_robot_imu_orange"><color rgba="0.95 0.45 0.05 1.0"/></material>
+      </visual>
+      <collision><geometry><box size="${' '.join(str(v) for v in imu['housing']['size'])}"/></geometry></collision>
+      <inertial>
+        <mass value="${imu['housing']['mass']}"/>
+        <inertia ixx="${imu['housing']['inertia']['ixx']}" ixy="0" ixz="0"
+                 iyy="${imu['housing']['inertia']['iyy']}" iyz="0"
+                 izz="${imu['housing']['inertia']['izz']}"/>
+      </inertial>
+    </link>
+    <joint name="${imu['joint_name']}" type="fixed">
+      <parent link="${imu['parent']}"/><child link="${imu['link_name']}"/>
+      <origin xyz="${' '.join(str(v) for v in imu['xyz'])}" rpy="${' '.join(str(v) for v in imu['rpy'])}"/>
+    </joint>
+    <gazebo reference="${imu['link_name']}">
+      <sensor name="imu_sensor" type="imu">
+        <topic>/ai_robot_internal/imu</topic>
+        <update_rate>${imu['update_rate_hz']}</update_rate>
+        <imu>
+          <angular_velocity>
+            <x><noise type="gaussian"><mean>0</mean><stddev>${imu['angular_velocity_noise_stddev']}</stddev></noise></x>
+            <y><noise type="gaussian"><mean>0</mean><stddev>${imu['angular_velocity_noise_stddev']}</stddev></noise></y>
+            <z><noise type="gaussian"><mean>0</mean><stddev>${imu['angular_velocity_noise_stddev']}</stddev></noise></z>
+          </angular_velocity>
+          <linear_acceleration>
+            <x><noise type="gaussian"><mean>0</mean><stddev>${imu['linear_acceleration_noise_stddev']}</stddev></noise></x>
+            <y><noise type="gaussian"><mean>0</mean><stddev>${imu['linear_acceleration_noise_stddev']}</stddev></noise></y>
+            <z><noise type="gaussian"><mean>0</mean><stddev>${imu['linear_acceleration_noise_stddev']}</stddev></noise></z>
+          </linear_acceleration>
+        </imu>
+        <always_on>true</always_on><visualize>true</visualize>
+      </sensor>
+    </gazebo>
+  </xacro:macro>
 </robot>

Commit message: feat(m4): 完成 W3 至 W8 整机集成验证

File: src/robot_core/ai_robot_description/urdf/ai_robot.urdf.xacro (robot description, xacro)
@@ -8,4 +8,5 @@
   <xacro:arg name="enable_imu" default="false"/>
   <xacro:arg name="controller_config" default=""/>
+  <xacro:arg name="controller_odom_topic" default="odom"/>
   <xacro:property name="model_config_path" value="$(arg model_config)"/>
   <xacro:property name="sensor_config_path" value="$(arg sensor_config)"/>
@@ -40,5 +41,8 @@
   </xacro:if>
   <xacro:if value="$(arg enable_control)">
-    <xacro:gazebo_control controller_config="$(arg controller_config)"/>
+    <xacro:gazebo_control
+      controller_config="$(arg controller_config)"
+      odom_topic="$(arg controller_odom_topic)"
+    />
   </xacro:if>
 </robot>

File: src/robot_core/ai_robot_description/urdf/macros/control.xacro (robot description, xacro)
@@ -1,5 +1,5 @@
 <?xml version="1.0"?>
 <robot xmlns:xacro="http://www.ros.org/wiki/xacro">
-  <xacro:macro name="gazebo_control" params="controller_config">
+  <xacro:macro name="gazebo_control" params="controller_config odom_topic">
     <ros2_control name="GazeboSimSystem" type="system">
       <hardware>
@@ -23,5 +23,5 @@
           <namespace>/robot</namespace>
           <remapping>diff_drive_base_controller/cmd_vel_unstamped:=controller_cmd_vel</remapping>
-          <remapping>diff_drive_base_controller/odom:=odom</remapping>
+          <remapping>diff_drive_base_controller/odom:=${odom_topic}</remapping>
           <remapping>tf:=/tf</remapping>
         </ros>
